Commit message: added stuff for gazebo

File: description/robot_arm.urdf.xacro (robot description, xacro)
@@ -1,10 +1,6 @@
 <?xml version="1.0"?>
 <robot xmlns:xacro="http://www.ros.org/wiki/xacro" name="robot">
-    <link name="world"></link>
-    <joint name="base_joint" type="fixed">
-        <origin xyz="1.5 1.0 0" rpy="0 0 0" />
-        <parent link="world" />
-        <child link="base_link" />
-    </joint>
+    <xacro:include filename="include.xacro" />
+    <link name="world" />
     <link name="base_link">
         <visual>
@@ -13,4 +9,5 @@
                 <box size="0.1 0.1 0.05" />
             </geometry>
+            <material name="white" />
         </visual>
         <collision>
@@ -20,10 +17,13 @@
             </geometry>
         </collision>
-        <inertial>
-            <mass value="1" />
+        <xacro:inertial_box mass="0.5" x="0.1" y="0.1" z="0.05">
             <origin rpy="0 0 0" xyz="0 0 0" />
-            <inertia ixx="0.001" ixy="0" ixz="0" iyy="0.001" iyz="0" izz="0.001" />
-        </inertial>
+        </xacro:inertial_box>
     </link>
+    <joint name="base_joint" type="fixed">
+        <origin xyz="0 0 0" rpy="0 0 0" />
+        <parent link="world" />
+        <child link="base_link" />
+    </joint>
     <link name="base_plate">
         <visual>
@@ -32,4 +32,5 @@
             </geometry>
             <origin rpy="0 0 0" xyz="0 0 0.0025" />
+            <material name="white" />
         </visual>
         <collision>
@@ -39,9 +40,7 @@
             <origin rpy="0 0 0" xyz="0 0 0.0025" />
         </collision>
-        <inertial>
-            <mass value="1" />
+        <xacro:inertial_cylinder mass="0.5" length="0.005" radius="0.04">
             <origin rpy="0 0 0" xyz="0 0 0" />
-            <inertia ixx="1" ixy="0" ixz="0" iyy="1" iyz="0" izz="1" />
-        </inertial>
+        </xacro:inertial_cylinder>
     </link>
     <joint name="base_plate_to_base_link" type="revolute">
@@ -58,4 +57,5 @@
             </geometry>
             <origin rpy="0 0 0" xyz="0 0 0.025" />
+            <material name="white" />
         </visual>
         <collision>
@@ -65,9 +65,7 @@
             <origin rpy="0 0 0" xyz="0 0 0.025" />
         </collision>
-        <inertial>
-            <mass value="1" />
+        <xacro:inertial_box mass="0.5" x="0.025" y="0.04" z="0.05">
             <origin rpy="0 0 0" xyz="0 0 0" />
-            <inertia ixx="1" ixy="0" ixz="0" iyy="1" iyz="0" izz="1" />
-        </inertial>
+        </xacro:inertial_box>
     </link>
     <joint name="base_plate_to_attachment" type="fixed">
@@ -82,4 +80,5 @@
             </geometry>
             <origin rpy="-1.5707963 0 0" xyz="0 -0.05 0" />
+            <material name="white" />
         </visual>
         <collision>
@@ -89,9 +88,7 @@
             <origin rpy="-1.5707963 0 0" xyz="0 -0.05 0" />
         </collision>
-        <inertial>
-            <mass value="1" />
+        <xacro:inertial_box mass="0.5" x="0.025" y="0.04" z="0.125">
             <origin rpy="0 0 0" xyz="0 0 0" />
-            <inertia ixx="1" ixy="0" ixz="0" iyy="1" iyz="0" izz="1" />
-        </inertial>
+        </xacro:inertial_box>
     </link>
     <joint name="mid_arm_to_attachment" type="revolute">
@@ -108,4 +105,5 @@
             </geometry>
             <origin rpy="-1.5707963 0 0" xyz="0 -0.025 0" />
+            <material name="white" />
         </visual>
         <collision>
@@ -115,9 +113,7 @@
             <origin rpy="-1.5707963 0 0" xyz="0 -0.025 0" />
         </collision>
-        <inertial>
-            <mass value="1" />
+        <xacro:inertial_box mass="0.5" x="0.025" y="0.04" z="0.085">
             <origin rpy="0 0 0" xyz="0 0 0" />
-            <inertia ixx="1" ixy="0" ixz="0" iyy="1" iyz="0" izz="1" />
-        </inertial>
+        </xacro:inertial_box>
     </link>
     <joint name="top_arm_to_mid_arm" type="revolute">
@@ -128,33 +124,13 @@
         <child link="top_arm" />
     </joint>
-    <inertial>
-        <mass value="1" />
-        <origin rpy="0 0 0" xyz="0 0 0" />
-        <inertia ixx="1" ixy="0" ixz="0" iyy="1" iyz="0" izz="1" />
-    </inertial>
-    <gazebo reference="base_link">
-        <material>Gazebo/Red</material>
-    </gazebo>
-    <gazebo reference="base_plate">
-        <material>Gazebo/Red</material>
-    </gazebo>
-    <gazebo reference="base_plate_attachment">
-        <material>Gazebo/Red</material>
-    </gazebo>
-    <gazebo reference="mid_arm">
-        <material>Gazebo/Red</material>
-    </gazebo>
-    <gazebo reference="top_arm">
-        <material>Gazebo/Red</material>
-    </gazebo>
     <gazebo>
         <plugin name="gazebo_ros_joint_state_publisher"
             filename="libgazebo_ros_joint_state_publisher.so">
-            <update_rate>20</update_rate>
+            <update_rate>30</update_rate>
             <joint_name>base_plate_to_base_link</joint_name>
-            <joint_name>base_plate_to_attachment</joint_name>
             <joint_name>mid_arm_to_attachment</joint_name>
             <joint_name>top_arm_to_mid_arm</joint_name>
         </plugin>
     </gazebo>
+    <!-- <xacro:include filename="gazebo.xacro" /> -->
 </robot>
